File: hardware/KiCad_Project/AquaSense/AquaSense.kicad_sch (KiCad schematic)
At the start: 0 parts

Commit message: Create hierarchical schematic and complete USB-C power interface
Other:
- added sheet Debug_Programming (05_Debug_Programming.kicad_sch)
- added sheet ESP32_Module (03_ESP32_Module.kicad_sch)
- added sheet Power (01_Power.kicad_sch)
- added sheet Sensor_Interfaces (04_Sensor_Interfaces.kicad_sch)
- added sheet User_Interface (06_User_Interface.kicad_sch)
- added sheet nRF52832_Core (02_nRF52832_Core.kicad_sch)
- title: (none) -> AquaSense
