File: hardware/KiCad_Project/AquaSense/02_nRF52832_Core.kicad_sch (KiCad schematic)
At the start: 0 parts

Commit message: Complete MCU core Schematic
Parts:
- added D2: LED, symbol Device:LED
- added J2: Conn_ARM_JTAG_SWD_10, Connector_PinHeader_1.27mm:PinHeader_2x05_P1.27mm_Vertical, symbol Connector:Conn_ARM_JTAG_SWD_10
- added J3: Conn_01x04, symbol Connector_Generic:Conn_01x04
- added R5: 10k, symbol Device:R
- added R6: 330, symbol Device:R
- added SW1: SW_Push, symbol Switch:SW_Push
- added U3: E73-2G4M04S-52832, RF_Module:E73-2G4M04S, symbol RF_Module:E73-2G4M04S-52832
Connections:
- new net: D2.2 (A), R6.2
- new net DS18B20_IO: U3.20 (AIN3/P0.05)
- new net GND: D2.1 (K), J2.3 (GND), J2.5 (GND), J2.9 (GNDDetect), J3.2 (Pin_2), SW1.1, U3.0 (GND), U3.1 (GND), U3.15 (GND), U3.2 (GND), U3.42 (GND), U3.43 (GND)
- new net RESET: J2.10 (~{RESET}), R5.2, SW1.2, U3.36 (P0.21/~{RESET})
- new net SWDCLK: J2.4 (SWCLK/TCK), U3.37 (SWDCLK)
- new net SWDIO: J2.2 (SWDIO/TMS), U3.38 (SWDIO)
- new net Status_LED: R6.1, U3.21 (P0.06)
- new net TDS_ADC: U3.18 (AIN1/P0.03)
- new net Turbidity_ADC: U3.19 (AIN2/P0.04)
- new net UART_RX: J3.4 (Pin_4), U3.24 (NFC1/P0.09)
- new net UART_TX: J3.3 (Pin_3), U3.23 (P0.08)
- new net VCC_3V3: J2.1 (VTref), J3.1 (Pin_1), R5.1, U3.16 (VCC)
- new net pH_ADC: U3.17 (AIN0/P0.02)
- no-connect marks 0 -> 29
Other:
- note added: "Connector Header"
- note added: "Debug"
- note added: "MCU"
