File: hardware/KiCad_Project/AquaSense/04_Sensor_Interfaces.kicad_sch (KiCad schematic)
At the start: 0 parts

Commit message: Complete Sensor Interface Schematic
Parts:
- added C5, C6, C7: 100nF, symbol Device:C
- added J4: J_pH, symbol Connector_Generic:Conn_01x03
- added J5: J_TDS, symbol Connector_Generic:Conn_01x03
- added J6: J_TURB, symbol Connector_Generic:Conn_01x03
- added J7: J_DS18B20, symbol Connector_Generic:Conn_01x03
- added R11, R7, R9: 100, symbol Device:R
- added R13: 4.7k, symbol Device:R
Connections:
- new net: J5.3 (Pin_3), R9.1
- new net: J6.3 (Pin_3), R11.1
- new net: J4.3 (Pin_3), R7.1
- new net DS18B20_IO: J7.3 (Pin_3), R13.1
- new net GND: C5.2, C6.2, C7.2, J4.2 (Pin_2), J5.2 (Pin_2), J6.2 (Pin_2), J7.2 (Pin_2)
- new net TDS_ADC: C6.1, R9.2
- new net Turbidity_ADC: C7.1, R11.2
- new net VCC_3V3: J4.1 (Pin_1), J5.1 (Pin_1), J6.1 (Pin_1), J7.1 (Pin_1), R13.2
- new net pH_ADC: C5.1, R7.2
